File: Proyecto_Bioimpedancia.sch (KiCad schematic (older format))
At the start: 69 parts, among them J1 Jumper, J2 Jumper, J3 Jumper_Calibration, J4 Jumper, J5 Jumper, J6 Jumper, P1 SD_LAPIZ, P10 RS-232, P11 SOURCE_2, P12 RESET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

Commit message: PCB BIO mejorada con puertos I2C y capacitor para el puerto DTR del programador FTDI
Parts:
- removed P10: RS-232, Socket_Strips:Socket_Strip_Straight_1x03_Pitch2.54mm, symbol CONN_01X03
- removed P6: I2C_1, Socket_Strips:Socket_Strip_Straight_1x02_Pitch2.54mm, symbol CONN_01X02
- removed P7: I2C_2, Socket_Strips:Socket_Strip_Straight_1x02_Pitch2.54mm, symbol CONN_01X02
- added C14: 0,1uF, Capacitors_SMD:C_0805_HandSoldering, symbol 0,1uF
- added P10: RS-232, Socket_Strips:Socket_Strip_Straight_1x04_Pitch2.54mm, symbol CONN_01X04
- added P6: CONN_02X04, Socket_Strips:Socket_Strip_Straight_2x04_Pitch2.54mm, symbol CONN_02X04
Connections:
- net AGND: now also P10.1 (P1)
- net RESET: now also C14.2
- net RXD: now also P10.3 (P3)
- net SCL_R: now also P6.1 (P1), P6.3 (P3), P6.5 (P5), P6.7 (P7)
- net SDA_R: now also P6.2 (P2), P6.4 (P4), P6.6 (P6), P6.8 (P8)
- net TXD: now also P10.2 (P2)
- new net: C14.1, P10.4 (P4)

Commit message: Revert "PCB BIO mejorada con puertos I2C y capacitor para el puerto DTR del programador FTDI"
This reverts commit 0fb084b6cb4dcbd826a5771fbeb8258d6327cef0.
Parts:
- removed C14: 0,1uF, Capacitors_SMD:C_0805_HandSoldering, symbol 0,1uF
- removed P10: RS-232, Socket_Strips:Socket_Strip_Straight_1x04_Pitch2.54mm, symbol CONN_01X04
- removed P6: CONN_02X04, Socket_Strips:Socket_Strip_Straight_2x04_Pitch2.54mm, symbol CONN_02X04
- added P10: RS-232, Socket_Strips:Socket_Strip_Straight_1x03_Pitch2.54mm, symbol CONN_01X03
- added P6: I2C_1, Socket_Strips:Socket_Strip_Straight_1x02_Pitch2.54mm, symbol CONN_01X02
- added P7: I2C_2, Socket_Strips:Socket_Strip_Straight_1x02_Pitch2.54mm, symbol CONN_01X02
Connections:
- net AGND: now also P10.1 (P1)
- net RXD: now also P10.3 (P3)
- net SCL_R: now also P6.2 (P2), P7.2 (P2)
- net SDA_R: now also P6.1 (P1), P7.1 (P1)
- net TXD: now also P10.2 (P2)
