File: Proyecto_Bioimpedancia.sch (KiCad schematic (older format))
At the start: 74 parts, among them J1 Jumper, J2 Jumper, J3 Jumper_Calibration, J4 Jumper, J5 Jumper, J6 Jumper, P1 SD_LAPIZ, P10 UNIVERSAL_PINS, P11 SOURCE_2, P12 RESET, P13 POWER, P14 BIO_OUT1, P15 GND_REGULATOR, P16 BIO_OUT2, P17 TOR_1, P18 TOR_2, P19 TOR_3, P2 GPIO, P20 TOR_4, P3 SOURCE_3, P4 SERIAL_VIRTUAL, P5 ENCODER, P6 I2C, P7 CONN_01X04, P8 SOURCE_1, P9 SPI, SW1 SW_PUSH, U1 AD8606, U2 ADG819, U3 Atmega328PA, U4 LD1117S50TR, Y1 XRCHA_16M

Commit message: Led Prueba Blink Añadido
Parts:
- added D5: Led_Small_Reg, LEDs:LED_0805, symbol Led_Small_Reg
- added R18: 1K, Resistors_SMD:R_0805_HandSoldering, symbol 1K
Connections:
- net AGND: now also D5.1 (K)
- net REG2_1: now also R18.2
- new net: D5.2 (A), R18.1
Other:
- note added: "Arreglo Blink"
Changed lines of the file:
@@
 U 1 1 5912ECD8
 P 5500 1350
-F 0 "R10" H 5530 1370 50  0000 L CNN
+F 0 "R10" V 5570 1280 50  0000 L CNN
 F 1 "RCAL" V 5400 1250 50  0000 L CNN
 F 2 "Resistors_SMD:R_0805_HandSoldering" H 5500 1350 50  0001 C CNN
@@
 NoConn ~ 7720 6070
 NoConn ~ 7310 6070
+Wire Notes Line
+	9080 5730 9080 6410
+Wire Notes Line
+	9080 6410 10090 6410
+Wire Notes Line
+	9080 5730 10090 5730
+Text Notes 9330 5810 0    39   ~ 0
+Arreglo Blink
+$Comp
+L Led_Small_Reg D5
+U 1 1 59D6CCBE
+P 9350 6080
+F 0 "D5" H 9300 6205 50  0000 L CNN
+F 1 "Led_Small_Reg" H 9110 5970 50  0000 L CNN
+F 2 "LEDs:LED_0805" H 9200 6105 50  0001 C CNN
+F 3 "" V 9350 6080 50  0000 C CNN
+F 4 "475-1410-2-ND" H 9400 6305 60  0001 C CNN "LED GREEN DIFFUSED 0805 SMD"
+	1    9350 6080
+	1    0    0    -1
+$EndComp
+$Comp
+L 1K R18
+U 1 1 59D75A52
+P 9620 6080
+F 0 "R18" V 9780 6060 50  0000 L CNN
+F 1 "1K" V 9710 6060 50  0000 L CNN
+F 2 "Resistors_SMD:R_0805_HandSoldering" H 9550 6000 50  0001 C CNN
+F 3 "" H 9650 6100 50  0000 C CNN
+F 4 "RMCF0805FT1K00TR-ND" H 9750 6200 39  0001 C CNN "RES SMD 1K OHM 1% 1/8W 0805"
+	1    9620 6080
+	0    -1   -1   0
+$EndComp
+Wire Wire Line
+	9450 6080 9520 6080
+Wire Wire Line
+	9720 6080 9830 6080
+Wire Wire Line
+	9250 6080 9150 6080
+Wire Wire Line
+	9150 6080 9150 5940
+Text Label 9150 5940 0    39   ~ 0
+AGND
+Text Label 9830 6080 0    39   ~ 0
+REG2_1
+Wire Notes Line
+	10090 5730 10090 6410
 $EndSCHEMATC

Commit message: Capacitores de Cristal 0402 cambiados
Parts:
- C5, C6: footprint Capacitors_SMD:C_0805_HandSoldering -> Capacitors_SMD:C_0402
Changed lines of the file:
@@
 	4100 1800 4250 1800
 Wire Wire Line
-	8570 1160 7920 1160
+	7920 1160 8570 1160
 Wire Wire Line
 	7920 1060 8220 1060
@@
 	3210 6660 3460 6660
 Wire Wire Line
-	10780 4770 10420 4770
+	10420 4770 10780 4770
 Wire Wire Line
 	9380 4720 9380 4800
@@
 	1910 7130 1910 7200
 Wire Wire Line
-	1500 6970 1500 6980
+	1500 6980 1500 6970
 Wire Wire Line
 	700  6980 1640 6980
@@
 F 0 "C5" H 4160 7130 50  0000 L CNN
 F 1 "8pF" H 4160 6980 50  0000 L CNN
-F 2 "Capacitors_SMD:C_0805_HandSoldering" H 4060 7030 50  0001 C CNN
+F 2 "Capacitors_SMD:C_0402" H 4060 7030 50  0001 C CNN
 F 3 "" H 4160 7130 50  0000 C CNN
 F 4 "399-1113-2-ND" H 4260 7230 39  0001 C CNN "CAP CER 22PF 50V C0G/NP0 0805"
@@
 F 0 "C6" H 4860 7130 50  0000 L CNN
 F 1 "8pF" H 4860 6980 50  0000 L CNN
-F 2 "Capacitors_SMD:C_0805_HandSoldering" H 4760 7030 50  0001 C CNN
+F 2 "Capacitors_SMD:C_0402" H 4760 7030 50  0001 C CNN
 F 3 "" H 4860 7130 50  0000 C CNN
 F 4 "399-1113-2-ND" H 4960 7230 39  0001 C CNN "CAP CER 22PF 50V C0G/NP0 0805"
