File: BIO_Respaldo.kicad_pcb (KiCad board)
At the start: 2 copper layers, 100 x 100 mm, 70 parts, among them J1 Jumper, J2 Jumper, J3 Jumper_Calibration, J4 Jumper, J5 Jumper, J6 Jumper, P1 SD_LAPIZ, P10 UNIVERSAL_PINS, P11 SOURCE_2, P12 RESET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

Commit message: PCB version final
Parts:
- removed P10: UNIVERSAL_PINS, Huellas:Universal_Path_80_Pins
Routing:
- net /AGND: vias 93 -> 91
- net (no net): track 0.00 -> 0.01 mm, vias 2 -> 0
Other:
- board text removed: "UNIVERSAL_PINS"
